File: ProtoCV.kicad_pcb (KiCad board)
At the start: 2 copper layers, 100 x 100 mm, 142 parts, among them J1 AudioJack2_SwitchT, J10 Conn_01x01_Male, J11 Conn_01x05_Male, J12 Conn_01x09_Male, J13 AudioJack2_SwitchT, J14 AudioJack2_SwitchT, J15 AudioJack2_SwitchT, J16 AudioJack2_SwitchT, J17 AudioJack2_SwitchT, J18 AudioJack2_SwitchT, J19 AudioJack2_SwitchT, J2 AudioJack2_SwitchT, J20 AudioJack2_SwitchT, J21 Conn_01x01_Male, J22 Conn_01x01_Male, J23 Conn_01x01_Male, J24 Conn_01x01_Male, J25 Conn_01x01_Male, J26 Conn_01x01_Male, J27 Conn_01x01_Male, J28 Conn_01x01_Male, J29 Conn_01x01_Male, J3 AudioJack2_SwitchT, J30 Conn_01x01_Male, J4 AudioJack2_SwitchT, J5 AudioJack2_SwitchT, J6 AudioJack2_SwitchT, J7 AudioJack2_SwitchT, J8 AudioJack2_SwitchT, J9 Conn_02x05_Odd_Even, Q1 BC847, Q2 BC847, Q3 BC847, Q4 BC847, Q5 BC847, Q6 BC847, Q7 BC847, Q8 BC847, U1 OPA4192, U2 OPA4192, U3 ADC80508Z, U4 R-78E3.3-0.5, U5 LD2981ABU33TR, U6 74AHCT244, U7 L7805

Commit message: Branding.
Other:
- board text added: "+12V"
- board text added: "-12V"
- board text added: "Marangisto 2020"
- board text added: "ProtoCV"
- board text added: "Rev A"
Changed lines of the file:
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@@
   (general
     (thickness 1.6)
-    (drawings 4)
+    (drawings 10)
     (tracks 901)
     (zones 0)
@@
     (tags resistor)
     (attr smd)
-    (fp_text reference R27 (at 0 -1.43) (layer F.SilkS)
+    (fp_text reference R27 (at 0 -1.27) (layer F.SilkS)
       (effects (font (size 1 1) (thickness 0.15)))
     )
@@
     (tags "PowerDI diode vishay")
     (attr smd)
-    (fp_text reference D2 (at 0 -2) (layer F.SilkS)
+    (fp_text reference D2 (at 0 -1.651) (layer F.SilkS)
       (effects (font (size 1 1) (thickness 0.15)))
     )
@@
     (tags "PowerDI diode vishay")
     (attr smd)
-    (fp_text reference D1 (at 0 -2) (layer F.SilkS)
+    (fp_text reference D1 (at 0 -1.905) (layer F.SilkS)
       (effects (font (size 1 1) (thickness 0.15)))
     )
@@
     )
   )
+  (gr_text "Marangisto 2020" (at 183.642 122.555) (layer F.SilkS)
+    (effects (font (size 1 1) (thickness 0.15)))
+  )
+  (gr_text "Rev A" (at 168.148 54.229) (layer F.SilkS)
+    (effects (font (size 1 1) (thickness 0.15)))
+  )
+  (gr_text ProtoCV (at 117.729 60.198) (layer F.SilkS)
+    (effects (font (size 4 3) (thickness 0.5)))
+  )
+  (gr_text +12V (at 161.544 55.626 90) (layer F.SilkS)
+    (effects (font (size 1 1) (thickness 0.15)))
+  )
+  (gr_text "-12V\n" (at 146.177 55.499 90) (layer F.SilkS)
+    (effects (font (size 1 1) (thickness 0.15)))
+  )
+  (gr_line (start 147.193 52.832) (end 147.193 57.912) (layer F.SilkS) (width 0.3))
   (gr_line (start 100 150) (end 100 50) (layer Edge.Cuts) (width 0.05))
   (gr_line (start 200 150) (end 100 150) (layer Edge.Cuts) (width 0.05))
